File: led_frame.sch (KiCad schematic (older format))
At the start: 130 parts

Commit message: layout
Parts:
- removed D? (x30): NeoPixel_THT, symbol NeoPixel_THT
- removed R? (x2): 100, symbol R
- added R10: R_PHOTO, Discret:R1, symbol R_PHOTO
- added R9: 10K, Resistors_THT:R_Axial_DIN0207_L6.3mm_D2.5mm_P7.62mm_Horizontal, symbol R
- added U2: MIC_MAX4466, led_frame:MAX4466_adafruit, symbol MIC_MAX4466
- added U3: StepDown_D24V50F5, led_frame:D24V50F5_pololu, symbol StepDown_D24V50F5
- D1, D10, D100, D101, D102, D105, D106, D107, D108, D109, D11, D110, D113, D114, D115, D116, D117, D118, D12, D13, D14, D17, D18, D19, D2, D20, D21, D22, D25, D26, D27, D28, D29, D3, D30, D33, D34, D35, D36, D37, D38, D4, D41, D42, D43, D44, D45, D46, D49, D5, D50, D51, D52, D53, D54, D57, D58, D59, D6, D60, D61, D62, D65, D66, D67, D68, D69, D70, D73, D74, D75, D76, D77, D78, D81, D82, D83, D84, D85, D86, D89, D9, D90, D91, D92, D93, D94, D97, D98, D99: renamed from D?; footprint (none) -> LEDs:LED_D5.0mm-4
- J1: renamed from J?; footprint (none) -> Connectors_Terminal_Blocks:TerminalBlock_Pheonix_PT-3.5mm_2pol
- R1, R2, R3, R4, R5, R6: renamed from R?; footprint (none) -> Resistors_THT:R_Axial_DIN0207_L6.3mm_D2.5mm_P7.62mm_Horizontal
- U1: renamed from U?; footprint (none) -> led_frame:teensy-lc
Connections:
- net at U1.15: now also U2.3 (OUT)
- net at U1.16: now also R10.2, R9.1
- net at U1.24 (3.3V): now also R10.1, U2.1 (VCC)
- net at U1.25 (GND): now also D1.2 (GND), D10.2 (GND), D100.2 (GND), D101.2 (GND), D102.2 (GND), D105.2 (GND), D106.2 (GND), D107.2 (GND), D108.2 (GND), D109.2 (GND), D11.2 (GND), D110.2 (GND), D113.2 (GND), D114.2 (GND), D115.2 (GND), D116.2 (GND), D117.2 (GND), D118.2 (GND), D12.2 (GND), D13.2 (GND), D14.2 (GND), D17.2 (GND), D18.2 (GND), D19.2 (GND), D2.2 (GND), D20.2 (GND), D21.2 (GND), D22.2 (GND), D25.2 (GND), D26.2 (GND), D27.2 (GND), D28.2 (GND), D29.2 (GND), D3.2 (GND), D30.2 (GND), D33.2 (GND), D34.2 (GND), D35.2 (GND), D36.2 (GND), D37.2 (GND), D38.2 (GND), D4.2 (GND), D41.2 (GND), D42.2 (GND), D43.2 (GND), D44.2 (GND), D45.2 (GND), D46.2 (GND), D49.2 (GND), D5.2 (GND), D50.2 (GND), D51.2 (GND), D52.2 (GND), D53.2 (GND), D54.2 (GND), D57.2 (GND), D58.2 (GND), D59.2 (GND), D6.2 (GND), D60.2 (GND), D61.2 (GND), D62.2 (GND), D65.2 (GND), D66.2 (GND), D67.2 (GND), D68.2 (GND), D69.2 (GND), D70.2 (GND), D73.2 (GND), D74.2 (GND), D75.2 (GND), D76.2 (GND), D77.2 (GND), D78.2 (GND), D81.2 (GND), D82.2 (GND), D83.2 (GND), D84.2 (GND), D85.2 (GND), D86.2 (GND), D89.2 (GND), D9.2 (GND), D90.2 (GND), D91.2 (GND), D92.2 (GND), D93.2 (GND), D94.2 (GND), D97.2 (GND), D98.2 (GND), D99.2 (GND), R9.2, U2.2 (GNC), U3.4 (GND)
- net at U1.26 (VIN): now also D1.3 (VDD), D10.3 (VDD), D100.3 (VDD), D101.3 (VDD), D102.3 (VDD), D105.3 (VDD), D106.3 (VDD), D107.3 (VDD), D108.3 (VDD), D109.3 (VDD), D11.3 (VDD), D110.3 (VDD), D113.3 (VDD), D114.3 (VDD), D115.3 (VDD), D116.3 (VDD), D117.3 (VDD), D118.3 (VDD), D12.3 (VDD), D13.3 (VDD), D14.3 (VDD), D17.3 (VDD), D18.3 (VDD), D19.3 (VDD), D2.3 (VDD), D20.3 (VDD), D21.3 (VDD), D22.3 (VDD), D25.3 (VDD), D26.3 (VDD), D27.3 (VDD), D28.3 (VDD), D29.3 (VDD), D3.3 (VDD), D30.3 (VDD), D33.3 (VDD), D34.3 (VDD), D35.3 (VDD), D36.3 (VDD), D37.3 (VDD), D38.3 (VDD), D4.3 (VDD), D41.3 (VDD), D42.3 (VDD), D43.3 (VDD), D44.3 (VDD), D45.3 (VDD), D46.3 (VDD), D49.3 (VDD), D5.3 (VDD), D50.3 (VDD), D51.3 (VDD), D52.3 (VDD), D53.3 (VDD), D54.3 (VDD), D57.3 (VDD), D58.3 (VDD), D59.3 (VDD), D6.3 (VDD), D60.3 (VDD), D61.3 (VDD), D62.3 (VDD), D65.3 (VDD), D66.3 (VDD), D67.3 (VDD), D68.3 (VDD), D69.3 (VDD), D70.3 (VDD), D73.3 (VDD), D74.3 (VDD), D75.3 (VDD), D76.3 (VDD), D77.3 (VDD), D78.3 (VDD), D81.3 (VDD), D82.3 (VDD), D83.3 (VDD), D84.3 (VDD), D85.3 (VDD), D86.3 (VDD), D89.3 (VDD), D9.3 (VDD), D90.3 (VDD), D91.3 (VDD), D92.3 (VDD), D93.3 (VDD), D94.3 (VDD), D97.3 (VDD), D98.3 (VDD), D99.3 (VDD), U3.5 (OUT)
- net at J1.1: now also U3.2 (VIN)
- net at J1.2: now also U3.3 (GND)
Other:
- moved on the sheet: D1, D10, D100, D101, D102, D105, D106, D107, D108, D109, D11, D110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
